File: layouts/default/default.kicad_pcb (KiCad board)
At the start: 2 copper layers, 5 parts

Commit message: frozen
Connections:
- U1 pad 10: hv -> gnd

Commit message: updated SPI interface
Parts:
- C1: value 100nF ±10% 50V X7R -> 10µF ±10% 25V X5R
Connections:
- net cs renamed NSS
- net hv renamed VCC
- net miso renamed MISO
- net mosi renamed MOSI
- net sck renamed SCK
Changed lines of the file:
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@@
     (net 0 "")
     (net 1 "TXEN")
-    (net 2 "miso")
+    (net 2 "MISO")
     (net 3 "BUSY")
-    (net 4 "hv")
-    (net 5 "sck")
-    (net 6 "mosi")
+    (net 4 "VCC")
+    (net 5 "SCK")
+    (net 6 "MOSI")
     (net 7 "NRST")
     (net 8 "DIO2")
@@
     (net 10 "ANT")
     (net 11 "gnd")
-    (net 12 "cs")
+    (net 12 "NSS")
     (net 13 "DIO")
     (footprint "atopile:R0402-56259e"
@@
             (size 0.57 0.54)
             (layers "F.Cu" "F.Mask" "F.Paste")
-            (net 4 "hv")
+            (net 4 "VCC")
         )
         (pad "2" smd rect
@@
             )
         )
-        (property "Value" "100nF ±10% 50V X7R"
+        (property "Value" "10µF ±10% 25V X5R"
             (at 0 0 0)
             (layer "F.Fab")
@@
             )
         )
-        (property "LCSC" "C49678"
-            (at 0 0 0)
-            (layer "User.9")
-            (hide yes)
-            (effects
-                (font
-                    (size 0.125 0.125)
-                    (thickness 0.01875)
-                )
-            )
-        )
-        (property "Partnumber" "CC0805KRX7R9BB104"
-            (at 0 0 0)
-            (layer "User.9")
-            (hide yes)
-            (effects
-                (font
-                    (size 0.125 0.125)
-                    (thickness 0.01875)
-                )
-            )
-        )
-        (property "Manufacturer" "YAGEO"
-            (at 0 0 0)
-            (layer "User.9")
-            (hide yes)
-            (effects
-                (font
-                    (size 0.125 0.125)
-                    (thickness 0.01875)
-                )
-            )
-        )
-        (property "JLCPCB description" "50V 100nF X7R ±10% 0805 Multilayer Ceramic Capacitors MLCC - SMD/SMT ROHS"
-            (at 0 0 0)
-            (layer "User.9")
-            (hide yes)
-            (effects
-                (font
-                    (size 0.125 0.125)
-                    (thickness 0.01875)
-                )
-            )
-        )
-        (property "PARAM_capacitance" "{\"type\": \"Quantity_Interval_Disjoint\", \"data\": {\"intervals\": {\"type\": \"Numeric_Interval_Disjoint\", \"data\": {\"intervals\": [{\"type\": \"Numeric_Interval\", \"data\": {\"min\": 9e-08, \"max\": 1.1e-07}}]}}, \"unit\": \"farad\"}}"
-            (at 0 0 0)
-            (layer "User.9")
-            (hide yes)
-            (effects
-                (font
-                    (size 0.125 0.125)
-                    (thickness 0.01875)
-                )
-            )
-        )
-        (property "PARAM_temperature_coefficient" "{\"type\": \"EnumSet\", \"data\": {\"elements\": [{\"name\": \"X7R\"}], \"enum\": {\"name\": \"TemperatureCoefficient\", \"values\": {\"Y5V\": 1, \"Z5U\": 2, \"X7S\": 3, \"X5R\": 4, \"X6R\": 5, \"X7R\": 6, \"X8R\": 7, \"C0G\": 8}}}}"
-            (at 0 0 0)
-            (layer "User.9")
-            (hide yes)
-            (effects
-                (font
-                    (size 0.125 0.125)
-                    (thickness 0.01875)
-                )
-            )
-        )
-        (property "PARAM_max_voltage" "{\"type\": \"Quantity_Set_Discrete\", \"data\": {\"intervals\": {\"type\": \"Numeric_Interval_Disjoint\", \"data\": {\"intervals\": [{\"type\": \"Numeric_Interval\", \"data\": {\"min\": 50.0, \"max\": 50.0}}]}}, \"unit\": \"volt\"}}"
+        (property "LCSC" "C15850"
+            (at 0 0 0)
+            (layer "User.9")
+            (hide yes)
+            (effects
+                (font
+                    (size 0.125 0.125)
+                    (thickness 0.01875)
+                )
+            )
+        )
+        (property "Partnumber" "CL21A106KAYNNNE"
+            (at 0 0 0)
+            (layer "User.9")
+            (hide yes)
+            (effects
+                (font
+                    (size 0.125 0.125)
+                    (thickness 0.01875)
+                )
+            )
+        )
+        (property "Manufacturer" "Samsung Electro-Mechanics"
+            (at 0 0 0)
+            (layer "User.9")
+            (hide yes)
+            (effects
+                (font
+                    (size 0.125 0.125)
+                    (thickness 0.01875)
+                )
+            )
+        )
+        (property "JLCPCB description" "25V 10uF X5R ±10% 0805 Multilayer Ceramic Capacitors MLCC - SMD/SMT ROHS"
+            (at 0 0 0)
+            (layer "User.9")
+            (hide yes)
+            (effects
+                (font
+                    (size 0.125 0.125)
+                    (thickness 0.01875)
+                )
+            )
+        )
+        (property "PARAM_capacitance" "{\"type\": \"Quantity_Interval_Disjoint\", \"data\": {\"intervals\": {\"type\": \"Numeric_Interval_Disjoint\", \"data\": {\"intervals\": [{\"type\": \"Numeric_Interval\", \"data\": {\"min\": 8.999999985e-06, \"max\": 1.1000000015e-05}}]}}, \"unit\": \"farad\"}}"
+            (at 0 0 0)
+            (layer "User.9")
+            (hide yes)
+            (effects
+                (font
+                    (size 0.125 0.125)
+                    (thickness 0.01875)
+                )
+            )
+        )
+        (property "PARAM_temperature_coefficient" "{\"type\": \"EnumSet\", \"data\": {\"elements\": [{\"name\": \"X5R\"}], \"enum\": {\"name\": \"TemperatureCoefficient\", \"values\": {\"Y5V\": 1, \"Z5U\": 2, \"X7S\": 3, \"X5R\": 4, \"X6R\": 5, \"X7R\": 6, \"X8R\": 7, \"C0G\": 8}}}}"
+            (at 0 0 0)
+            (layer "User.9")
+            (hide yes)
+            (effects
+                (font
+                    (size 0.125 0.125)
+                    (thickness 0.01875)
+                )
+            )
+        )
+        (property "PARAM_max_voltage" "{\"type\": \"Quantity_Set_Discrete\", \"data\": {\"intervals\": {\"type\": \"Numeric_Interval_Disjoint\", \"data\": {\"intervals\": [{\"type\": \"Numeric_Interval\", \"data\": {\"min\": 25.0, \"max\": 25.0}}]}}, \"unit\": \"volt\"}}"
             (at 0 0 0)
             (layer "User.9")
@@
             (size 1.41 1.35)
             (layers "F.Cu" "F.Mask" "F.Paste")
-            (net 4 "hv")
+            (net 4 "VCC")
         )
         (pad "2" smd rect
@@
             (size 0.79 0.54)
             (layers "F.Cu" "F.Mask" "F.Paste")
-            (net 4 "hv")
+            (net 4 "VCC")
         )
         (pad "2" smd rect
@@
             (size 1.8 0.9)
             (layers "F.Cu" "F.Mask" "F.Paste")
-            (net 4 "hv")
+            (net 4 "VCC")
         )
         (pad "10" smd rect
@@
             (size 1.8 0.9)
             (layers "F.Cu" "F.Mask" "F.Paste")
-            (net 2 "miso")
+            (net 2 "MISO")
         )
         (pad "17" smd rect
@@
             (size 1.8 0.9)
             (layers "F.Cu" "F.Mask" "F.Paste")
-            (net 6 "mosi")
+            (net 6 "MOSI")
         )
         (pad "18" smd rect
@@
             (size 1.8 0.9)
             (layers "F.Cu" "F.Mask" "F.Paste")
-            (net 5 "sck")
+            (net 5 "SCK")
         )
         (pad "19" smd rect
@@
             (size 1.8 0.9)
             (layers "F.Cu" "F.Mask" "F.Paste")
-            (net 12 "cs")
+            (net 12 "NSS")
         )
         (pad "20" smd rect
@@
             (size 0.57 0.54)
             (layers "F.Cu" "F.Mask" "F.Paste")
-            (net 4 "hv")
+            (net 4 "VCC")
         )
         (pad "2" smd rect
